Commit message: import a new model with steering wheel --------------------------------------------------- How to use: terminal 1: 	cd motorcycle_ws 	catkin_make 	source devel/setup.bash 	roslaunch motorcycle_gz motorcycle_world.launch 	press space in Gazebo terminal 2:(crtl+shift+T) 	source devel/setup.bash 	roslaunch motorcycle_gz motorcycle.launch

File: src/motorcycle_description_direction/motorcycle_description/urdf/motorcycle_description.urdf (robot description, URDF)
Before this commit: robot motorcycle_description, 3 links, 2 joints
Links:
- added link direction_link, mass 0006154.7356109696; collision mesh filename=package://motorcycle_description/meshes/direction_link.STL; visual mesh filename=package://motorcycle_description/meshes/direction_link.STL
- link base_link: mass 0289701.940057169 -> 0286167.648321881
Joints:
- added joint direction_joint: type revolute, parent base_link, child direction_link, origin xyz=0.058 0 -0.01 rpy=0 0 -0.033503, axis 0 0 -1, limit lower=-0.5235 upper=0.5235 effort=0 velocity=0
- joint wheel_back_joint: origin xyz=-0.048172 0 -0.020493 rpy=0 0 0 -> xyz=-0.028 0 -0.028 rpy=0 0 0
- joint wheel_front_joint: axis 0 1 0 -> -0.033748 -0.99943 0; origin xyz=0.037828 0 -0.020493 rpy=0 0 0 -> xyz=0 0 -0.018 rpy=0 0 0.033503; parent base_link -> direction_link

Commit message: read direction parameter and control it, but some pysical parameter need to be real velocity keep add state friction and moving friction

File: src/motorcycle_description_direction/motorcycle_description/urdf/motorcycle_description.urdf (robot description, URDF)
Before this commit: robot motorcycle_description, 4 links, 3 joints
Joints:
- joint direction_joint: axis 0 0 -1 -> 0 0 1; limit lower=-0.5235 upper=0.5235 effort=0 velocity=0 -> lower=-1 upper=1 effort=0 velocity=0
