Commit message: Enter force:2,000,000 in gazebo interface, to go straight

File: src/motorcycle_description/urdf/motorcycle_description.urdf (robot description, URDF)
Before this commit: robot motorcycle_description, 4 links, 3 joints
Joints:
- joint FrontFork_Joint: limit lower=0 upper=0 effort=0 velocity=0 -> lower=${-pi*0.9} upper=${pi*0.9} effort=1000 velocity=100; type continuous -> revolute

Commit message: ROS_Control Go Straight by Force with Code without Balance Control

File: src/motorcycle_description/urdf/motorcycle_description.urdf (robot description, URDF)
Before this commit: robot motorcycle_description, 4 links, 3 joints
Joints:
- joint Bwheel_Joint: limit lower=0 upper=0 effort=0 velocity=0 -> (none)

Commit message: rewrite loadparameter_force.cpp[publish] motorcycle_force.cpp[subscribe publish]

File: src/motorcycle_description/urdf/motorcycle_description.urdf (robot description, URDF)
Before this commit: robot motorcycle_description, 4 links, 3 joints
Joints:
- joint FrontFork_Joint: limit lower=${-pi*0.9} upper=${pi*0.9} effort=1000 velocity=100 -> lower=${-pi*0.8} upper=${pi*0.8} effort=10000 velocity=10000

Commit message: subscribe velocity and have pid template

File: src/motorcycle_description/urdf/motorcycle_description.urdf (robot description, URDF)
Before this commit: robot motorcycle_description, 4 links, 3 joints
Joints:
- joint FrontFork_Joint: limit lower=${-pi*0.8} upper=${pi*0.8} effort=10000 velocity=10000 -> lower=${-pi*0.5} upper=${pi*0.5} effort=10000000000 velocity=10000000000

Commit message: subscribe imu quaternion

File: src/motorcycle_description/urdf/motorcycle_description.urdf (robot description, URDF)
Before this commit: robot motorcycle_description, 4 links, 3 joints
Links:
- link Body_Link: mass 7211369.76127266 -> 85
- link Bwheel_Link: mass 1392324.96652693 -> 5
- link Direction_Link: mass 0550171.42922688 -> 5
- link Fwheel_Link: mass 1392325.39502733 -> 5

Commit message: Add PID on Steer

File: src/motorcycle_description/urdf/motorcycle_description.urdf (robot description, URDF)
Before this commit: robot motorcycle_description, 4 links, 3 joints
Links:
- link Body_Link: mass 85 -> 65
- link Direction_Link: mass 5 -> 25
Joints:
- joint FrontFork_Joint: limit lower=${-pi*0.5} upper=${pi*0.5} effort=10000000000 velocity=10000000000 -> lower=${-45*pi/180} upper=${45*pi/180} effort=10000000000 velocity=10000000000

Commit message: go straight (change mass, p:1 i:0.05 d:0)

File: src/motorcycle_description/urdf/motorcycle_description.urdf (robot description, URDF)
Before this commit: robot motorcycle_description, 4 links, 3 joints
Links:
- link Body_Link: mass 65 -> 45
- link Direction_Link: mass 25 -> 45
